Commit message: converted to 3 wheel robot and added position, velocity, balanced PID with reasonable tuning

File: src/mybot_description/urdf/mybot.xacro (robot description, xacro)
@@ -7,16 +7,15 @@
   <xacro:include filename="$(find mybot_description)/urdf/macros.xacro" />
   <link name='chassis'>
-    <pose>0 0 0.4 0 0 0</pose>
-    <inertial>
-      <mass value="15.0"/>
-      <origin xyz="0.0 0 0.6" rpy=" 0 0 0"/>
-      <inertia
-          ixx="0.1" ixy="0" ixz="0"
-          iyy="0.1" iyz="0"
-          izz="0.1"
+    <inertial>
+      <mass value="75.0"/>
+      <origin xyz="0.0 0 0.0" rpy=" 0 0 0"/>
+      <inertia
+          ixx="0.3125" ixy="0" ixz="0"
+          iyy="4.25" iyz="0"
+          izz="4.0625"
       />
     </inertial>
     <collision name='collision'>
-      <origin xyz="0 0 0.5" rpy=" 0 0 0"/>
+      <origin xyz="0 0 0" rpy=" 0 0 0"/>
       <geometry>
         <box size=".8 .2 .1"/>
@@ -24,5 +23,5 @@
     </collision>
     <visual name='chassis_visual'>
-      <origin xyz="0 0 0.5" rpy=" 0 0 0"/>
+      <origin xyz="0 0 0" rpy=" 0 0 0"/>
       <geometry>
         <box size=".8 .2 .1"/>
@@ -30,21 +29,11 @@
     </visual>
     <collision name='support1_collision'>
-      <origin xyz="-0.375 0 0.25" rpy=" 0 0 0"/>
-      <geometry>
-        <box size="0.05 0.2 0.4" />
-      </geometry>
-      <surface>
-        <friction>
-          <ode>
-            <mu>0</mu>
-            <mu2>0</mu2>
-            <slip1>1.0</slip1>
-            <slip2>1.0</slip2>
-          </ode>
-        </friction>
-      </surface>
+      <origin xyz="-0.375 0 -0.25" rpy=" 0 0 0"/>
+      <geometry>
+        <box size="0.05 0.2 0.4" />
+      </geometry>
     </collision>
     <visual name='chassis_visual'>
-      <origin xyz="-0.375 0 0.25" rpy=" 0 0 0"/>
+      <origin xyz="-0.375 0 -0.25" rpy=" 0 0 0"/>
       <geometry>
         <box size="0.05 0.2 0.4" />
@@ -52,21 +41,11 @@
     </visual>
     <collision name='support2_collision'>
-      <origin xyz="0.375 0 0.25" rpy=" 0 0 0"/>
-      <geometry>
-        <box size="0.05 0.2 0.4" />
-      </geometry>
-      <surface>
-        <friction>
-          <ode>
-            <mu>0</mu>
-            <mu2>0</mu2>
-            <slip1>1.0</slip1>
-            <slip2>1.0</slip2>
-          </ode>
-        </friction>
-      </surface>
+      <origin xyz="0.375 0 -0.25" rpy=" 0 0 0"/>
+      <geometry>
+        <box size="0.05 0.2 0.4" />
+      </geometry>
     </collision>
     <visual name='chassis_visual'>
-      <origin xyz="0.375 0 0.25" rpy=" 0 0 0"/>
+      <origin xyz="0.375 0 -0.25" rpy=" 0 0 0"/>
       <geometry>
         <box size="0.05 0.2 0.4" />
@@ -81,4 +60,12 @@
         <cylinder radius="0.1" length="0.05"/>
       </geometry>
+      <surface>
+        <friction>
+          <ode>
+            <mu>200.0</mu>
+            <mu2>200</mu2>
+          </ode>
+        </friction>
+      </surface>
     </collision>
     <visual name="left_wheel_visual">
@@ -90,9 +77,9 @@
     <inertial>
       <origin xyz="0 0 0" rpy="0 1.5707 1.5707"/>
-      <mass value="5"/>
-      <inertia
-        ixx=".1" ixy="0.0" ixz="0.0"
-        iyy=".1" iyz="0.0"
-        izz=".1"/>
+      <mass value="0.5"/>
+      <inertia
+        ixx=".00135" ixy="0.0" ixz="0.0"
+        iyy=".00135" iyz="0.0"
+        izz=".0025"/>
     </inertial>
   </link>
@@ -104,4 +91,12 @@
         <cylinder radius="0.1" length="0.05"/>
       </geometry>
+      <surface>
+        <friction>
+          <ode>
+            <mu>200.0</mu>
+            <mu2>200</mu2>
+          </ode>
+        </friction>
+      </surface>
     </collision>
     <visual name="left_wheel_rear_visual">
@@ -113,9 +108,9 @@
     <inertial>
       <origin xyz="0 0 0" rpy="0 1.5707 1.5707"/>
-      <mass value="5"/>
-      <inertia
-        ixx=".1" ixy="0.0" ixz="0.0"
-        iyy=".1" iyz="0.0"
-        izz=".1"/>
+      <mass value="0.5"/>
+      <inertia
+        ixx=".00135" ixy="0.0" ixz="0.0"
+        iyy=".00135" iyz="0.0"
+        izz=".0025"/>
     </inertial>
   </link>
@@ -123,22 +118,30 @@
     <!--origin xyz="0.1 -0.13 0.1" rpy="0 1.5707 1.5707"/-->
     <collision name="collision">
-      <origin xyz="0 0 0" rpy="0 1.5707 1.5707"/>
-      <geometry>
-        <cylinder radius="0.1" length="0.05"/>
-      </geometry>
+      <origin xyz="0 0 0" rpy="0 -1.5707 -1.5707"/>
+      <geometry>
+        <cylinder radius="0.01" length="0.05"/>
+      </geometry>
+      <surface>
+        <friction>
+          <ode>
+            <mu>200.0</mu>
+            <mu2>200</mu2>
+          </ode>
+        </friction>
+      </surface>
     </collision>
     <visual name="right_wheel_visual">
-      <origin xyz="0 0 0" rpy="0 1.5707 1.5707"/>
-      <geometry>
-        <cylinder radius="0.1" length="0.05"/>
-      </geometry>
-    </visual>
-    <inertial>
-      <origin xyz="0 0 0" rpy="0 1.5707 1.5707"/>
-      <mass value="5"/>
-      <inertia
-        ixx=".1" ixy="0.0" ixz="0.0"
-        iyy=".1" iyz="0.0"
-        izz=".1"/>
+      <origin xyz="0 0 0" rpy="0 -1.5707 -1.5707"/>
+      <geometry>
+        <cylinder radius="0.01" length="0.05"/>
+      </geometry>
+    </visual>
+    <inertial>
+      <origin xyz="0 0 0" rpy="0 1.5707 1.5707"/>
+      <mass value="0.5"/>
+      <inertia
+        ixx=".00135" ixy="0.0" ixz="0.0"
+        iyy=".00135" iyz="0.0"
+        izz=".0025"/>
     </inertial>
   </link>
@@ -146,22 +149,30 @@
     <!--origin xyz="0.1 -0.13 0.1" rpy="0 1.5707 1.5707"/-->
     <collision name="collision">
-      <origin xyz="0 0 0" rpy="0 1.5707 1.5707"/>
-      <geometry>
-        <cylinder radius="0.1" length="0.05"/>
-      </geometry>
+      <origin xyz="0 0 0" rpy="0 -1.5707 -1.5707"/>
+      <geometry>
+        <cylinder radius="0.1" length="0.05"/>
+      </geometry>
+      <surface>
+        <friction>
+          <ode>
+            <mu>200.0</mu>
+            <mu2>200</mu2>
+          </ode>
+        </friction>
+      </surface>
     </collision>
     <visual name="right_wheel_rear_visual">
-      <origin xyz="0 0 0" rpy="0 1.5707 1.5707"/>
-      <geometry>
-        <cylinder radius="0.1" length="0.05"/>
-      </geometry>
-    </visual>
-    <inertial>
-      <origin xyz="0 0 0" rpy="0 1.5707 1.5707"/>
-      <mass value="5"/>
-      <inertia
-        ixx=".1" ixy="0.0" ixz="0.0"
-        iyy=".1" iyz="0.0"
-        izz=".1"/>
+      <origin xyz="0 0 0" rpy="0 -1.5707 -1.5707"/>
+      <geometry>
+        <cylinder radius="0.1" length="0.05"/>
+      </geometry>
+    </visual>
+    <inertial>
+      <origin xyz="0 0 0" rpy="0 1.5707 1.5707"/>
+      <mass value="0.5"/>
+      <inertia
+        ixx=".00135" ixy="0.0" ixz="0.0"
+        iyy=".00135" iyz="0.0"
+        izz=".0025"/>
     </inertial>
   </link>
@@ -184,11 +195,11 @@
       <mass value="0.0001"/>
       <inertia
-        ixx=".0001" ixy="0.0" ixz="0.0"
-        iyy=".0001" iyz="0.0"
-        izz=".0001"/>
+        ixx=".000001" ixy="0.0" ixz="0.0"
+        iyy=".000001" iyz="0.0"
+        izz=".000001"/>
     </inertial>
   </link>
   <joint type="fixed" name="imu_hinge">
-    <origin xyz="0 0 0.555" rpy="0 0 0"/>
+    <origin xyz="0 0 0.055" rpy="0 0 0"/>
     <!--origin xyz="0.1 -0.13 0" rpy="0 1.5707 1.5707"/-->
     <child link="imu_link"/>
@@ -199,46 +210,46 @@
   </joint>
   <joint type="continuous" name="left_wheel_hinge">
-    <origin xyz="0.375 0.12 .1" rpy="0 0 0"/>
+    <origin xyz="0.375 0.0 -0.4" rpy="0 0 0"/>
     <!--origin xyz="0.1 0.13 0" rpy="0 1.5707 1.5707"/-->
     <child link="left_wheel"/>
     <parent link="chassis"/>
     <axis xyz="0 1 0" rpy="0 0 0"/>
-    <limit effort="10000" velocity="1000"/>
-    <joint_properties damping="1.0" friction="1.0"/>
+    <limit effort="100" velocity="100"/>
+    <joint_properties damping="10.0" friction="10.0"/>
   </joint>
   <joint type="continuous" name="right_wheel_hinge">
-    <origin xyz="0.375 -0.12 0.1" rpy="0 0 0"/>
+    <origin xyz="0.375 -0.13 -0.4" rpy="0 0 0"/>
     <!--origin xyz="0.1 -0.13 0" rpy="0 1.5707 1.5707"/-->
     <child link="right_wheel"/>
     <parent link="chassis"/>
     <axis xyz="0 1 0" rpy="0 0 0"/>
-    <limit effort="10000" velocity="1000"/>
-    <joint_properties damping="1.0" friction="1.0"/>
+    <limit effort="100" velocity="100"/>
+    <joint_properties damping="10.0" friction="10.0"/>
   </joint>
   <joint type="continuous" name="left_wheel_rear_hinge">
-    <origin xyz="-0.375 0.12 0.1" rpy="0 0 0"/>
+    <origin xyz="-0.375 0.13 -0.4" rpy="0 0 0"/>
     <!--origin xyz="0.1 0.13 0" rpy="0 1.5707 1.5707"/-->
     <child link="left_wheel_rear"/>
     <parent link="chassis"/>
     <axis xyz="0 1 0" rpy="0 0 0"/>
-    <limit effort="10000" velocity="1000"/>
-    <joint_properties damping="1.0" friction="1.0"/>
+    <limit effort="100" velocity="100"/>
+    <joint_properties damping="10.0" friction="0.0"/>
   </joint>
   <joint type="continuous" name="right_wheel_rear_hinge">
-    <origin xyz="-0.375 -0.12 0.1" rpy="0 0 0"/>
+    <origin xyz="-0.375 -0.13 -0.4" rpy="0 0 0"/>
     <!--origin xyz="0.1 -0.13 0" rpy="0 1.5707 1.5707"/-->
     <child link="right_wheel_rear"/>
     <parent link="chassis"/>
     <axis xyz="0 1 0" rpy="0 0 0"/>
-    <limit effort="10000" velocity="1000"/>
-    <joint_properties damping="1.0" friction="1.0"/>
+    <limit effort="100" velocity="100"/>
+    <joint_properties damping="10.0" friction="0.0"/>
   </joint>
   <transmission name="tran_LF">
     <type>transmission_interface/SimpleTransmission</type>
     <joint name="left_wheel_hinge">
-      <hardwareInterface>hardware_interface/VelocityJointInterface</hardwareInterface>
+      <hardwareInterface>hardware_interface/EffortJointInterface</hardwareInterface>
     </joint>
     <actuator name="motor_LF">
-      <hardwareInterface>hardware_interface/VelocityJointInterface</hardwareInterface>
+      <hardwareInterface>hardware_interface/EffortJointInterface</hardwareInterface>
       <mechanicalReduction>1</mechanicalReduction>
     </actuator>
@@ -247,8 +258,8 @@
     <type>transmission_interface/SimpleTransmission</type>
     <joint name="right_wheel_hinge">
-      <hardwareInterface>hardware_interface/VelocityJointInterface</hardwareInterface>
+      <hardwareInterface>hardware_interface/EffortJointInterface</hardwareInterface>
     </joint>
     <actuator name="motor_RF">
-      <hardwareInterface>hardware_interface/VelocityJointInterface</hardwareInterface>
+      <hardwareInterface>hardware_interface/EffortJointInterface</hardwareInterface>
       <mechanicalReduction>1</mechanicalReduction>
     </actuator>
@@ -257,8 +268,8 @@
     <type>transmission_interface/SimpleTransmission</type>
     <joint name="left_wheel_rear_hinge">
-      <hardwareInterface>hardware_interface/VelocityJointInterface</hardwareInterface>
+      <hardwareInterface>hardware_interface/EffortJointInterface</hardwareInterface>
     </joint>
     <actuator name="motor_LR">
-      <hardwareInterface>hardware_interface/VelocityJointInterface</hardwareInterface>
+      <hardwareInterface>hardware_interface/EffortJointInterface</hardwareInterface>
       <mechanicalReduction>1</mechanicalReduction>
     </actuator>
@@ -267,8 +278,8 @@
     <type>transmission_interface/SimpleTransmission</type>
     <joint name="right_wheel_rear_hinge">
-      <hardwareInterface>hardware_interface/VelocityJointInterface</hardwareInterface>
+      <hardwareInterface>hardware_interface/EffortJointInterface</hardwareInterface>
     </joint>
     <actuator name="motor_RR">
-      <hardwareInterface>hardware_interface/VelocityJointInterface</hardwareInterface>
+      <hardwareInterface>hardware_interface/EffortJointInterface</hardwareInterface>
       <mechanicalReduction>1</mechanicalReduction>
     </actuator>
